File: corne-cherry/pcb/corne-cherry.kicad_sch (KiCad schematic)
At the start: 120 parts, among them J1 MJ-4PP-9, J2 OLED, J3 LED, P1 i2c-pin, P2 i2c-pin, SW1 SW_PUSH, SW10 SW_PUSH, SW11 SW_PUSH, SW12 SW_PUSH, SW13 SW_PUSH, SW14 SW_PUSH, SW15 SW_PUSH, SW16 SW_PUSH, SW17 SW_PUSH, SW18 SW_PUSH, SW19 SW_PUSH, SW2 SW_PUSH, SW20 SW_PUSH, SW21 SW_PUSH, SW22 SW_PUSH, SW23 SW_PUSH, SW24 SW_PUSH, SW25 SW_PUSH, SW26 SW_PUSH, SW3 SW_PUSH, SW4 SW_PUSH, SW5 SW_PUSH, SW6 SW_PUSH, SW7 SW_PUSH, SW8 SW_PUSH, SW9 SW_PUSH, U1 ProMicro, U3 D, U5 D

Commit message: WIP refonte Rili : chantier KiCad + pipeline tripwire
- Schéma/PCB corne-cherry en cours de refonte ESP32/nRF24 (travail en cours,
  DRC assumé au-dessus de l'ancien état : baseline ratchet réalignée sur la
  réalité du chantier — 814 erreurs DRC, 175 warnings ; objectif zéro en fin
  de refonte)
- Pipeline anti-régression tripwire : scripts/check.sh, kicad-check.sh,
  hooks git + Claude Code, CI GitHub Actions, CLAUDE.md
- Bibliothèques locales : footprints (MaeLid, PMW3360, nice-nano, key…),
  symboles mae.kicad_sym, fp-lib-table, fichiers rescue
- .gitignore : réparation (marqueurs de conflit committés par erreur),
  ignore des locks KiCad et du dump fournisseur JC-ESP32P4-M3-C6 (350 Mo)

Co-Authored-By: Claude Fable 5 <noreply@anthropic.com>
Claude-Session: https://claude.ai/code/session_01RACBjiS4NRTWA7TWVi4mtR
Parts:
- removed J2: OLED, kbd:OLED, symbol Connector_Generic:Conn_01x04
- removed J3: LED, kbd:StripLED_rev, symbol Connector_Generic:Conn_01x03
- removed JP1: (no value), kbd:JPC2, symbol corne-cherry-rescue:Jumper-Device
- removed JP2, JP3, JP4, JP5, JP6, JP7, JP8, JP9: (no value), kbd:Jumper, symbol corne-cherry-rescue:Jumper_NO_Small-Device
- removed L1, L10, L11, L12, L13, L14, L15, L16, L17, L18, L19, L2, L20, L21, L28, L29, L3, L30, L31, L32, L4, L5, L6, L7, L8, L9: SK6812MINI, EKR82-footprint:SK6812MINI_rev, symbol corne-cherry-rescue:SK6812MINI-kbd-corne-cherry-rescue
- removed L22, L23: SK6812MINI, EKR82-footprint:SK6812MINI_underglow_rev, symbol corne-cherry-rescue:SK6812MINI-kbd-corne-cherry-rescue
- removed L24, L25, L26, L27, L33: SK6812MINI, EKR82-footprint:SK6812MINI_underglow_rev, symbol rouge_gorge:SK6812MINI-SMD
- removed RSW1: SW_PUSH, kbd:ResetSW, symbol corne-cherry-rescue:SW_PUSH-kbd-corne-cherry-rescue
- removed U1: ProMicro, kbd:ProMicro_v2, symbol corne-cherry-rescue:ProMicro-kbd-corne-cherry-rescue
- added R3, R4: 100R, Resistor_SMD:R_0603_1608Metric_Pad0.98x0.95mm_HandSolder, symbol Device:R
- R1, R2: value R -> 100R; footprint kbd:R -> Resistor_SMD:R_0603_1608Metric_Pad0.98x0.95mm_HandSolder
Connections:
- net VCC: no longer R1.1, R2.1
- net data: now also J1.B, P2.1 (Pin_1)
- net row0: now also R4.1; no longer D1.1 (K), D2.1 (K), D23.1 (K), D3.1 (K), D4.1 (K), D5.1 (K), D6.1 (K)
- net row1: now also R3.1; no longer D10.1 (K), D11.1 (K), D12.1 (K), D24.1 (K), D7.1 (K), D8.1 (K), D9.1 (K)
- net row2: now also R2.1; no longer D13.1 (K), D14.1 (K), D15.1 (K), D16.1 (K), D17.1 (K), D18.1 (K)
- net row3: now also R1.1; no longer D19.1 (K), D20.1 (K), D21.1 (K), D22.1 (K), U3.1 (K), U5.1 (K)
- net SCL: no longer names the net of R2.2
- net SCL: now also D13.1 (K), D14.1 (K), D15.1 (K), D16.1 (K), D17.1 (K), D18.1 (K)
- net SDA: no longer names the net of R1.2
- net SDA: now also D19.1 (K), D20.1 (K), D21.1 (K), D22.1 (K), U3.1 (K), U5.1 (K)
- new net: D1.1 (K), D2.1 (K), D23.1 (K), D3.1 (K), D4.1 (K), D5.1 (K), D6.1 (K), R4.2
- new net: D10.1 (K), D11.1 (K), D12.1 (K), D24.1 (K), D7.1 (K), D8.1 (K), D9.1 (K), R3.2
- no-connect marks 4 -> 0
Other:
- moved on the sheet: D1, D10, D11, D12, D13, D14, D15, D16, D17, D18, D19, D2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
