File: rili/pcb/usb_right.kicad_sch (KiCad schematic)
At the start: 4 parts, among them J403 USB_C_Receptacle_USB2.0_16P, U402 USBLC6-2SC6

Commit message: layout v2 : carte routée — PCB↔schéma réconciliés, BOM LCSC, TVS matrice, DRC 990→24
- réconciliation PCB↔schéma en une passe : 105 empreintes remariées (matrice ×2,
  module P4), 54 périmées supprimées, ~140 importées par F8 ; footprint TRRS
  MJ-4PP-9_rev3 créé (pads mappés de l'ancien design fonctionnel)
- placement : moitié droite générée au miroir exact du pré-placement gauche
  (axe x=188.46048), trous de montage symétrisés, origine de grille sur l'axe
- protection ESD matrice : 22 SD05C-01F (un par ligne, côté switchs des 100R,
  validés par partition de netlist) ; PWR_FLAG +5V_D réparé
- BOM LCSC dans les propriétés des symboles (32 composants : réfs, liens,
  notes d'achat) + annexe courses complète au plan v2 ; connecteur trackpad
  corrigé (ZIF Hirose FH12-6S-0.5SH, réf MNT Reform)
- règles JLCPCB (planchers DRC + classes Default/Power re-branchées v2),
  passage 4 couches, routage complet des deux moitiés
- gerbers v1 corne-cherry retirés (obsolètes)
- baselines tripwire re-référencées : DRC 990→24 erreurs / 208→17 warnings,
  ERC 0 erreur / 200 warnings (53 fantômes headless documentés)

Co-Authored-By: Claude Fable 5 <noreply@anthropic.com>
Claude-Session: https://claude.ai/code/session_01GfX5RmekmQi78Dm37qsT4Z
Parts:
- J7: renamed from J403; footprint (none) -> Connector_USB:USB_C_Receptacle_HRO_TYPE-C-31-M-12; LCSC (none) -> C165948; Lien (none) -> https://lcsc.com/product-detail/C165948.html
- U15: renamed from U402; LCSC (none) -> C7519; Lien (none) -> https://lcsc.com/product-detail/C7519.html
- renumbered R416 to R51, R417 to R53
Connections:
- no-connect marks 4 -> 2
