File: rili/pcb/p4.kicad_sch (KiCad schematic)
At the start: 16 parts, among them J6 Micro_SD_Card, U15 AMS1117-3.3, U6 ESP32P4_QFN104

Commit message: schéma v2 COMPLET : les deux moitiés — ERC 0 erreur
Architecture finale (brainstorm + nuit de réflexion, décision Mae) :
asymétrie d'origine confirmée — UN seul coffre.
- Gauche (s3/bat/usb/p4) : S3 + matrice + trackpad TPS43 + alim 16340
  + USB-C + hub CH334R + coffre P4 (SD multi-ISO, PGP, prog-via-hub)
- Droite (right/bat_right/usb_right, NOUVELLES feuilles) : S3 + matrice
  + écran Sharp + alim 16340 propre + USB-C simple (USBLC6 direct, sans hub)

Génération scriptée (make_droite/make_right_rails/cleanup, scratchpad) :
copies s3→right (refs +200) et bat→bat_right (refs +300, rails +BATT_D/
VSYS_D/+3.3V_D), usb→usb_right (refs +400, hub/P4/prog retirés, USBLC6
→ D±_s3_d, +5V_D), rails gauche/droite séparés (GND seul commun, physique
via TRRS), populate tranché (écran→droite, trackpad→gauche), feuille
Matrix retirée (matrice droite incluse dans right), droite.kicad_sch
remplacé par right.kicad_sch.

Validation : ERC projet 0 erreur ; nets droite bouclés de bout en bout
(+BATT_D→+3.3V_D→MCU, USB→USBLC6→MCU, jauge→GPIO13). Baseline warnings
re-référencée 125→164 (libs legacy doublées par la 2e moitié).

Prochaine phase : LAYOUT (réconciliation PCB↔schéma en une passe,
placement, routage, panneau sécable, DRC).

Co-Authored-By: Claude Fable 5 <noreply@anthropic.com>
Claude-Session: https://claude.ai/code/session_01GfX5RmekmQi78Dm37qsT4Z
Changed lines of the file:
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@@
-	)
-	(symbol
-		(lib_id "power:PWR_FLAG")
-		(at 163.83 173.99 0)
-		(unit 1)
-		(body_style 1)
-		(exclude_from_sim no)
-		(in_bom yes)
-		(on_board yes)
-		(in_pos_files yes)
-		(dnp no)
-		(fields_autoplaced yes)
-		(property "Reference" "#FLG01"
-			(at 163.83 172.085 0)
-			(hide yes)
-			(show_name no)
-			(do_not_autoplace no)
-			(effects
-				(font
-					(size 1.27 1.27)
-				)
-			)
-		)
-		(property "Value" "PWR_FLAG"
-			(at 163.83 168.91 0)
-			(show_name no)
-			(do_not_autoplace no)
-			(effects
-				(font
-					(size 1.27 1.27)
-				)
-			)
-		)
-		(property "Footprint" ""
-			(at 163.83 173.99 0)
-			(hide yes)
-			(show_name no)
-			(do_not_autoplace no)
-			(effects
-				(font
-					(size 1.27 1.27)
-				)
-			)
-		)
-		(property "Datasheet" ""
-			(at 163.83 173.99 0)
-			(hide yes)
-			(show_name no)
-			(do_not_autoplace no)
-			(effects
-				(font
-					(size 1.27 1.27)
-				)
-			)
-		)
-		(property "Description" "Special symbol for telling ERC where power comes from"
-			(at 163.83 173.99 0)
-			(hide yes)
-			(show_name no)
-			(do_not_autoplace no)
-			(effects
-				(font
-					(size 1.27 1.27)
-				)
-			)
-		)
-		(pin "1"
-		)
-		(instances
-			(project "niphar"
-				(path "/7138aad8-3c5f-41d0-9987-adc2f08f0576/002e7793-b48a-4c8b-b85c-dccde4948ad0"
-					(reference "#FLG01")
-					(unit 1)
-				)
-			)
-		)
 	)
 	(symbol

Commit message: layout v2 : carte routée — PCB↔schéma réconciliés, BOM LCSC, TVS matrice, DRC 990→24
- réconciliation PCB↔schéma en une passe : 105 empreintes remariées (matrice ×2,
  module P4), 54 périmées supprimées, ~140 importées par F8 ; footprint TRRS
  MJ-4PP-9_rev3 créé (pads mappés de l'ancien design fonctionnel)
- placement : moitié droite générée au miroir exact du pré-placement gauche
  (axe x=188.46048), trous de montage symétrisés, origine de grille sur l'axe
- protection ESD matrice : 22 SD05C-01F (un par ligne, côté switchs des 100R,
  validés par partition de netlist) ; PWR_FLAG +5V_D réparé
- BOM LCSC dans les propriétés des symboles (32 composants : réfs, liens,
  notes d'achat) + annexe courses complète au plan v2 ; connecteur trackpad
  corrigé (ZIF Hirose FH12-6S-0.5SH, réf MNT Reform)
- règles JLCPCB (planchers DRC + classes Default/Power re-branchées v2),
  passage 4 couches, routage complet des deux moitiés
- gerbers v1 corne-cherry retirés (obsolètes)
- baselines tripwire re-référencées : DRC 990→24 erreurs / 208→17 warnings,
  ERC 0 erreur / 200 warnings (53 fantômes headless documentés)

Co-Authored-By: Claude Fable 5 <noreply@anthropic.com>
Claude-Session: https://claude.ai/code/session_01GfX5RmekmQi78Dm37qsT4Z
Parts:
- J9: renamed from J6; Achat (none) -> Würth 693072010801 (Mouser/Farnell); Lien (none) -> https://www.mouser.com/ProductDetail/Wurth-Elektronik/69307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; Note achat (none) -> alt. LCSC TF-01A C91145 mais empreinte à changer
- U16: renamed from U6; Achat (none) -> module JC-ESP32P4-M3 V0.2 AliExpress/Taobao
- U17: renamed from U15; LCSC (none) -> C6186; Lien (none) -> https://lcsc.com/product-detail/C6186.html
- renumbered C8 to C14, C16 to C15, C15 to C16, C18 to C17, C17 to C18, R23 to R54, R24 to R55, R25 to R56, R26 to R57, R27 to R58, R28 to R59

Commit message: layout : panneau vertical 2 rails dans le dépôt + baseline chantier
Panneau 185×212 (droite tournée 180°, rails + 8 tabs mouse-bites) appliqué par
Mae, F8 des passifs unifiés. Baseline DRC re-référencée 24/19 → 36/26 (état
panneau, finitions DRC prévues : pistes près des lignes de rupture, vias de
maillage orphelins dans les bandes sans cuivre).

Co-Authored-By: Claude Fable 5 <noreply@anthropic.com>
Claude-Session: https://claude.ai/code/session_01GfX5RmekmQi78Dm37qsT4Z
Parts:
- C17: footprint Capacitor_SMD:C_0805_2012Metric_Pad1.18x1.45mm_HandSolder -> Capacitor_SMD:C_0603_1608Metric
Changed lines of the file:
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@@
 			)
 		)
-		(property "Footprint" "Capacitor_SMD:C_0805_2012Metric_Pad1.18x1.45mm_HandSolder"
+		(property "Footprint" "Capacitor_SMD:C_0603_1608Metric"
 			(at 191.4652 46.99 0)
 			(hide yes)

Commit message: review schéma : LDO S3 corrigé (pins SOT-89) + 8 valeurs — HT7833 en place
Revue 4 relecteurs parallèles avant commande, validée ligne à ligne sur la
netlist. BLOQUANT réparé : U20/U21 avaient le brochage SOT-23 du MCP1700 sur
des pastilles SOT-89 → entrée/sortie inversées pour tout LDO réel ; pins 2/3
échangés dans la déf, Value=HT7833 (C50936), F8 + reroutage des 2 zones par
Mae, pads vérifiés (1=GND 2=VIN 3=VOUT). Valeurs : bulk 3V3 C11/C12 et condos
LDO C23-C26 → 10µF (C15850), CHIP_PU P4 R54→10k C14→1µF. Baseline ERC 200→202
(lib_symbol_mismatch des défs LDO éditées). Validé par la revue : chaînes
batterie/charge/load-share, paires USB bout en bout, hub, prog P4 ×2 ports,
microSD IOMUX+pullups, strapping, nRF24, trackpad, 22 TVS matrice.

Co-Authored-By: Claude Fable 5 <noreply@anthropic.com>
Claude-Session: https://claude.ai/code/session_01GfX5RmekmQi78Dm37qsT4Z
Parts:
- C14: value 100nF -> 1uF; footprint Capacitor_SMD:C_0603_1608Metric -> Capacitor_SMD:C_0805_2012Metric_Pad1.18x1.45mm_HandSolder
- C16: value 22uF -> 10uF
- C17: footprint Capacitor_SMD:C_0603_1608Metric -> Capacitor_SMD:C_0603_1608Metric_Pad1.08x0.95mm_HandSolder
- R54: value 100k -> 10k; footprint Resistor_SMD:R_0603_1608Metric -> Resistor_SMD:R_0603_1608Metric_Pad0.98x0.95mm_HandSolder
- R55, R56, R57, R58, R59: footprint Resistor_SMD:R_0603_1608Metric -> Resistor_SMD:R_0603_1608Metric_Pad0.98x0.95mm_HandSolder
Changed lines of the file:
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@@
 			)
 		)
-		(property "Footprint" "Resistor_SMD:R_0603_1608Metric"
+		(property "Footprint" "Resistor_SMD:R_0603_1608Metric_Pad0.98x0.95mm_HandSolder"
 			(at 203.2 25.908 90)
 			(hide yes)
@@
 			)
 		)
-		(property "Value" "22uF"
+		(property "Value" "10uF"
 			(at 157.48 184.1499 0)
 			(show_name no)
@@
 			)
 		)
-		(property "Footprint" "Capacitor_SMD:C_0603_1608Metric"
+		(property "Footprint" "Capacitor_SMD:C_0603_1608Metric_Pad1.08x0.95mm_HandSolder"
 			(at 191.4652 46.99 0)
 			(hide yes)
@@
 			)
 		)
-		(property "Footprint" "Resistor_SMD:R_0603_1608Metric"
+		(property "Footprint" "Resistor_SMD:R_0603_1608Metric_Pad0.98x0.95mm_HandSolder"
 			(at 203.2 28.448 90)
 			(hide yes)
@@
 			)
 		)
-		(property "Value" "100k"
+		(property "Value" "10k"
 			(at 39.37 39.37 90)
 			(show_name no)
@@
 			)
 		)
-		(property "Footprint" "Resistor_SMD:R_0603_1608Metric"
+		(property "Footprint" "Resistor_SMD:R_0603_1608Metric_Pad0.98x0.95mm_HandSolder"
 			(at 39.37 41.148 90)
 			(hide yes)
@@
 			)
 		)
-		(property "Footprint" "Resistor_SMD:R_0603_1608Metric"
+		(property "Footprint" "Resistor_SMD:R_0603_1608Metric_Pad0.98x0.95mm_HandSolder"
 			(at 203.2 18.288 90)
 			(hide yes)
@@
 			)
 		)
-		(property "Footprint" "Resistor_SMD:R_0603_1608Metric"
+		(property "Footprint" "Resistor_SMD:R_0603_1608Metric_Pad0.98x0.95mm_HandSolder"
 			(at 203.2 20.828 90)
 			(hide yes)
@@
 			)
 		)
-		(property "Value" "100nF"
+		(property "Value" "1uF"
 			(at 44.196 40.64 0)
 			(show_name no)
@@
 			)
 		)
-		(property "Footprint" "Capacitor_SMD:C_0603_1608Metric"
+		(property "Footprint" "Capacitor_SMD:C_0805_2012Metric_Pad1.18x1.45mm_HandSolder"
 			(at 49.8348 39.37 0)
 			(hide yes)
@@
 			)
 		)
-		(property "Footprint" "Resistor_SMD:R_0603_1608Metric"
+		(property "Footprint" "Resistor_SMD:R_0603_1608Metric_Pad0.98x0.95mm_HandSolder"
 			(at 203.2 23.368 90)
 			(hide yes)
