File: rili/pcb/right.kicad_sch (KiCad schematic)
At the start: 101 parts, among them J2 Conn_02x03_Odd_Even, J4 Conn_01x05_Pin, J5 AudioJack4, SW11 SW_PUSH, SW13 SW_PUSH, SW16 SW_PUSH, SW18 SW_PUSH, SW2 SW_PUSH, SW20 SW_PUSH, SW22 SW_PUSH, SW23 SW_PUSH, SW25 SW_PUSH, SW28 SW_PUSH, SW29 SW_PUSH, SW32 SW_PUSH, SW34 SW_PUSH, SW36 SW_PUSH, SW37 SW_PUSH, SW39 SW_PUSH, SW4 SW_PUSH, SW42 SW_PUSH, SW44 SW_PUSH, SW46 SW_PUSH, SW48 SW_PUSH, SW50 SW_PUSH, SW51 SW_PUSH, SW6 SW_PUSH, SW7 SW_PUSH, SW9 SW_PUSH, U1 D, U10 SRV05-4, U11 SiP32431DR3, U4 D, U5 ESP32-S3-WROOM-1, U7 NRF24L01_Breakout

Commit message: review schéma : LDO S3 corrigé (pins SOT-89) + 8 valeurs — HT7833 en place
Revue 4 relecteurs parallèles avant commande, validée ligne à ligne sur la
netlist. BLOQUANT réparé : U20/U21 avaient le brochage SOT-23 du MCP1700 sur
des pastilles SOT-89 → entrée/sortie inversées pour tout LDO réel ; pins 2/3
échangés dans la déf, Value=HT7833 (C50936), F8 + reroutage des 2 zones par
Mae, pads vérifiés (1=GND 2=VIN 3=VOUT). Valeurs : bulk 3V3 C11/C12 et condos
LDO C23-C26 → 10µF (C15850), CHIP_PU P4 R54→10k C14→1µF. Baseline ERC 200→202
(lib_symbol_mismatch des défs LDO éditées). Validé par la revue : chaînes
batterie/charge/load-share, paires USB bout en bout, hub, prog P4 ×2 ports,
microSD IOMUX+pullups, strapping, nRF24, trackpad, 22 TVS matrice.

Co-Authored-By: Claude Fable 5 <noreply@anthropic.com>
Claude-Session: https://claude.ai/code/session_01GfX5RmekmQi78Dm37qsT4Z
Parts:
- C10, C4: footprint Capacitor_SMD:C_0805_2012Metric -> Capacitor_SMD:C_0805_2012Metric_Pad1.18x1.45mm_HandSolder
- C12: value 1uF -> 10uF; footprint Capacitor_SMD:C_0805_2012Metric -> Capacitor_SMD:C_1206_3216Metric_Pad1.33x1.80mm_HandSolder
- C2, C7: footprint Capacitor_SMD:C_0603_1608Metric -> Capacitor_SMD:C_0603_1608Metric_Pad1.08x0.95mm_HandSolder
- R1, R15, R17, R31, R33, R37, R38, R40: footprint Resistor_SMD:R_0603_1608Metric -> Resistor_SMD:R_0603_1608Metric_Pad0.98x0.95mm_HandSolder
- R10, R12, R13, R19, R22, R24, R26, R28, R3, R5, R8: value 100R -> 100
Changed lines of the file:
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@@
 			)
 		)
-		(property "Value" "100R"
+		(property "Value" "100"
 			(at 80.01 139.7 0)
 			(show_name no)
@@
 			)
 		)
-		(property "Footprint" "Resistor_SMD:R_0603_1608Metric"
+		(property "Footprint" "Resistor_SMD:R_0603_1608Metric_Pad0.98x0.95mm_HandSolder"
 			(at 72.39 49.022 90)
 			(hide yes)
@@
 			)
 		)
-		(property "Footprint" "Resistor_SMD:R_0603_1608Metric"
+		(property "Footprint" "Resistor_SMD:R_0603_1608Metric_Pad0.98x0.95mm_HandSolder"
 			(at 34.29 34.798 90)
 			(hide yes)
@@
 			)
 		)
-		(property "Value" "100R"
+		(property "Value" "100"
 			(at 34.29 177.8 90)
 			(show_name no)
@@
 			)
 		)
-		(property "Value" "100R"
+		(property "Value" "100"
 			(at 61.976 139.7 0)
 			(show_name no)
@@
 			)
 		)
-		(property "Footprint" "Resistor_SMD:R_0603_1608Metric"
+		(property "Footprint" "Resistor_SMD:R_0603_1608Metric_Pad0.98x0.95mm_HandSolder"
 			(at 227.33 74.168 90)
 			(hide yes)
@@
 			)
 		)
-		(property "Footprint" "Resistor_SMD:R_0603_1608Metric"
+		(property "Footprint" "Resistor_SMD:R_0603_1608Metric_Pad0.98x0.95mm_HandSolder"
 			(at 72.39 46.482 90)
 			(hide yes)
@@
 			)
 		)
-		(property "Value" "100R"
+		(property "Value" "100"
 			(at 53.34 140.9699 0)
 			(show_name no)
@@
 			)
 		)
-		(property "Value" "100R"
+		(property "Value" "100"
 			(at 34.29 162.56 90)
 			(show_name no)
@@
 			)
 		)
-		(property "Value" "1uF"
+		(property "Value" "10uF"
 			(at 267.462 58.674 0)
 			(show_name no)
@@
 			)
 		)
-		(property "Footprint" "Capacitor_SMD:C_0805_2012Metric"
+		(property "Footprint" "Capacitor_SMD:C_1206_3216Metric_Pad1.33x1.80mm_HandSolder"
 			(at 270.8148 57.15 0)
 			(hide yes)
@@
 			)
 		)
-		(property "Footprint" "Capacitor_SMD:C_0603_1608Metric"
+		(property "Footprint" "Capacitor_SMD:C_0603_1608Metric_Pad1.08x0.95mm_HandSolder"
 			(at 260.6548 57.15 0)
 			(hide yes)
@@
 			)
 		)
-		(property "Footprint" "Resistor_SMD:R_0603_1608Metric"
+		(property "Footprint" "Resistor_SMD:R_0603_1608Metric_Pad0.98x0.95mm_HandSolder"
 			(at 227.33 69.088 90)
 			(hide yes)
@@
 			)
 		)
-		(property "Footprint" "Capacitor_SMD:C_0805_2012Metric"
+		(property "Footprint" "Capacitor_SMD:C_0805_2012Metric_Pad1.18x1.45mm_HandSolder"
 			(at 269.5448 144.78 0)
 			(hide yes)
@@
 			)
 		)
-		(property "Footprint" "Resistor_SMD:R_0603_1608Metric"
+		(property "Footprint" "Resistor_SMD:R_0603_1608Metric_Pad0.98x0.95mm_HandSolder"
 			(at 198.12 52.578 90)
 			(hide yes)
@@
 			)
 		)
-		(property "Value" "100R"
+		(property "Value" "100"
 			(at 34.29 193.04 90)
 			(show_name no)
@@
 			)
 		)
-		(property "Value" "100R"
+		(property "Value" "100"
 			(at 115.57 139.7 0)
 			(show_name no)
@@
 			)
 		)
-		(property "Footprint" "Resistor_SMD:R_0603_1608Metric"
+		(property "Footprint" "Resistor_SMD:R_0603_1608Metric_Pad0.98x0.95mm_HandSolder"
 			(at 227.33 76.708 90)
 			(hide yes)
@@
 			)
 		)
-		(property "Footprint" "Capacitor_SMD:C_0603_1608Metric"
+		(property "Footprint" "Capacitor_SMD:C_0603_1608Metric_Pad1.08x0.95mm_HandSolder"
 			(at 44.7548 33.02 0)
 			(hide yes)
@@
 			)
 		)
-		(property "Value" "100R"
+		(property "Value" "100"
 			(at 133.35 139.954 0)
 			(show_name no)
@@
 			)
 		)
-		(property "Footprint" "Resistor_SMD:R_0603_1608Metric"
+		(property "Footprint" "Resistor_SMD:R_0603_1608Metric_Pad0.98x0.95mm_HandSolder"
 			(at 181.61 95.758 90)
 			(hide yes)
@@
 			)
 		)
-		(property "Value" "100R"
+		(property "Value" "100"
 			(at 34.29 208.28 90)
 			(show_name no)
@@
 			)
 		)
-		(property "Value" "100R"
+		(property "Value" "100"
 			(at 98.044 139.954 0)
 			(show_name no)
@@
 			)
 		)
-		(property "Value" "100R"
+		(property "Value" "100"
 			(at 155.702 139.7 0)
 			(show_name no)
@@
 			)
 		)
-		(property "Footprint" "Capacitor_SMD:C_0805_2012Metric"
+		(property "Footprint" "Capacitor_SMD:C_0805_2012Metric_Pad1.18x1.45mm_HandSolder"
 			(at 54.9148 33.02 0)
 			(hide yes)

Commit message: review : solde complet — Tip TRRS protégé, condos +BATT, prog P4 dégagée
- TVS Tip : canal 3 des SRV05 relié au Tip des deux jacks (net TIP_5V, validé
  netlist : jack.T + load switch OUT + SRV05 sans toucher LINK_5V_EN)
- C29/C30 : 10µF sur +BATT/+BATT_D près des TP4056, placés et routés par Mae
- R48/R49 supprimés par Mae (CH334R : pull-up RESET# interne 25k, mode
  sans-quartz XO flottant conforme datasheet, fuite batterie→hub éliminée)
- pistes JP1/JP2 (prog USB du P4) écartées de la zone GND : zéro violation
- nettoyage : no_connect orpheline de la dépose R48/R49
- DRC 36/26 → 17/22 (ménage de routage par Mae), ratchet enregistré

Décisions documentées : SD manipulée hors tension (pas de TVS SD), tables de
pins matrice réelles + conventions firmware en annexe du plan v2.

Co-Authored-By: Claude Fable 5 <noreply@anthropic.com>
Claude-Session: https://claude.ai/code/session_01GfX5RmekmQi78Dm37qsT4Z
Connections:
- net TIP_5V: now reaches J5.T, U11.1 (OUT)
- net TIP_5V: now also U10.3 (IO2)
- no-connect marks 8 -> 7
Changed lines of the file:
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@@
-	)
-	(no_connect
-		(at 364.49 86.36)
 	)
 	(no_connect
@@
 		)
 	)
+	(label "TIP_5V"
+		(at 364.49 86.36 0)
+		(effects
+			(font
+				(size 1.27 1.27)
+			)
+			(justify left bottom)
+		)
+	)
 	(label "col1"
 		(at 68.58 135.89 0)
@@
 		(effects
 			(font
+				(size 1.27 1.27)
+			)
+			(justify left bottom)
+		)
+	)
+	(label "TIP_5V"
+		(at 361.95 36.83 0)
+		(effects
+			(font
